File: hardware/led-cc-driver-mk-2.0.sch (EAGLE design)
At the start: 8 parts, among them Q1 2N3904, Q2 2N7000

Commit message: layout for cc driver and some dicking around with the rgb one
Parts:
- D1: device A_butts:DIODE-ZENERPTH-7.62MM -> A_butts:DIODE-ZENER7.62MM-PTH
- Q2: value 2N7000 -> FQP30N06L
- renumbered OUT to LED
Other:
- moved on the sheet: IN
Changed lines of the file:
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@@
 <parts>
 <part name="Q1" library="A_butts" deviceset="TRANSISTOR_NPN" device="TO-92-AMMO-EBC" value="2N3904"/>
-<part name="Q2" library="A_butts" deviceset="MOSFET-NCHANNEL" device="TO-220" value="2N7000"/>
+<part name="Q2" library="A_butts" deviceset="MOSFET-NCHANNEL" device="TO-220" value="FQP30N06L"/>
 <part name="R2" library="A_butts" deviceset="RESISTOR" device="PTH-AXIAL-10.16MM" value="Iset"/>
 <part name="SUPPLY2" library="A_butts" deviceset="VCC" device=""/>
 <part name="GND2" library="A_butts" deviceset="GND" device=""/>
 <part name="H1" library="A_butts" deviceset="HOLE" device="#2"/>
-<part name="OUT" library="A_butts" deviceset="M02" device="PTH" value="M02PTH"/>
+<part name="LED" library="A_butts" deviceset="M02" device="PTH" value="M02PTH"/>
 <part name="H2" library="A_butts" deviceset="HOLE" device="#2"/>
 <part name="IN" library="A_butts" deviceset="M03" device="PTH"/>
 <part name="SUPPLY1" library="A_butts" deviceset="VCC" device=""/>
 <part name="GND1" library="A_butts" deviceset="GND" device=""/>
-<part name="D1" library="A_butts" deviceset="DIODE-ZENER" device="PTH-7.62MM" value="10V"/>
+<part name="D1" library="A_butts" deviceset="DIODE-ZENER" device="7.62MM-PTH" value="10V"/>
 </parts>
 <sheets>
@@
 <instance part="SUPPLY2" gate="G$1" x="38.1" y="55.88"/>
 <instance part="GND2" gate="1" x="33.02" y="2.54"/>
-<instance part="H1" gate="G$1" x="63.5" y="53.34"/>
-<instance part="OUT" gate="G$1" x="50.8" y="48.26" rot="MR0"/>
-<instance part="H2" gate="G$1" x="68.58" y="53.34"/>
-<instance part="IN" gate="G$1" x="7.62" y="73.66"/>
-<instance part="SUPPLY1" gate="G$1" x="27.94" y="76.2"/>
-<instance part="GND1" gate="1" x="27.94" y="66.04"/>
+<instance part="H1" gate="G$1" x="7.62" y="40.64"/>
+<instance part="LED" gate="G$1" x="50.8" y="48.26" rot="MR0"/>
+<instance part="H2" gate="G$1" x="12.7" y="40.64"/>
+<instance part="IN" gate="G$1" x="7.62" y="53.34"/>
+<instance part="SUPPLY1" gate="G$1" x="27.94" y="55.88"/>
+<instance part="GND1" gate="1" x="27.94" y="45.72"/>
 <instance part="D1" gate="G$1" x="10.16" y="17.78" rot="R90"/>
 </instances>
@@
 <wire x1="38.1" y1="53.34" x2="38.1" y2="55.88" width="0.1524" layer="91"/>
 <wire x1="38.1" y1="53.34" x2="40.64" y2="53.34" width="0.1524" layer="91"/>
-<pinref part="OUT" gate="G$1" pin="2"/>
+<pinref part="LED" gate="G$1" pin="2"/>
 </segment>
 <segment>
 <pinref part="IN" gate="G$1" pin="2"/>
 <pinref part="SUPPLY1" gate="G$1" pin="VCC"/>
-<wire x1="15.24" y1="73.66" x2="27.94" y2="73.66" width="0.1524" layer="91"/>
-<wire x1="27.94" y1="73.66" x2="27.94" y2="76.2" width="0.1524" layer="91"/>
+<wire x1="15.24" y1="53.34" x2="27.94" y2="53.34" width="0.1524" layer="91"/>
+<wire x1="27.94" y1="53.34" x2="27.94" y2="55.88" width="0.1524" layer="91"/>
 </segment>
 </net>
@@
 <pinref part="IN" gate="G$1" pin="1"/>
 <pinref part="GND1" gate="1" pin="GND"/>
-<wire x1="15.24" y1="71.12" x2="27.94" y2="71.12" width="0.1524" layer="91"/>
-<wire x1="27.94" y1="71.12" x2="27.94" y2="68.58" width="0.1524" layer="91"/>
+<wire x1="15.24" y1="50.8" x2="27.94" y2="50.8" width="0.1524" layer="91"/>
+<wire x1="27.94" y1="50.8" x2="27.94" y2="48.26" width="0.1524" layer="91"/>
 </segment>
 </net>
@@
 <segment>
 <pinref part="IN" gate="G$1" pin="3"/>
-<wire x1="17.78" y1="76.2" x2="15.24" y2="76.2" width="0.1524" layer="91"/>
-<label x="17.78" y="76.2" size="1.27" layer="95" xref="yes"/>
+<wire x1="17.78" y1="55.88" x2="15.24" y2="55.88" width="0.1524" layer="91"/>
+<label x="17.78" y="55.88" size="1.27" layer="95" xref="yes"/>
 </segment>
 <segment>
@@
 <net name="N$4" class="0">
 <segment>
-<pinref part="OUT" gate="G$1" pin="1"/>
+<pinref part="LED" gate="G$1" pin="1"/>
 <pinref part="Q2" gate="G$1" pin="D"/>
 <wire x1="40.64" y1="50.8" x2="38.1" y2="50.8" width="0.1524" layer="91"/>
