File: hardware/rgb-led-cc-driver-mk-1.0.sch (EAGLE design)
At the start: 18 parts, among them IC1 TINY85-20-DIP, J1 AVR_SPI_PRG_6PTH_INLINE_I2C, Q1 2N3904, Q2 IRLZ14PBF, Q3 2N3904, Q4 IRLZ14PBF, Q5 2N3904, Q6 IRLZ14PBF

Commit message: layout for cc driver and some dicking around with the rgb one
Parts:
- D1, D2, D3: device A_butts:DIODE-ZENERPTH-7.62MM -> A_butts:DIODE-ZENER10.16MM-PTH
- Q2, Q4, Q6: value IRLZ14PBF -> FQP30N06L
- R1: device A_butts:RESISTORPTH-AXIAL-6.35MM -> A_butts:RESISTORPTH-AXIAL-10.16MM
Changed lines of the file:
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@@
 <parts>
 <part name="Q1" library="A_butts" deviceset="TRANSISTOR_NPN" device="TO-92-AMMO-EBC" value="2N3904"/>
-<part name="Q2" library="A_butts" deviceset="MOSFET-NCHANNEL" device="TO-220" value="IRLZ14PBF"/>
+<part name="Q2" library="A_butts" deviceset="MOSFET-NCHANNEL" device="TO-220" value="FQP30N06L"/>
 <part name="R2" library="A_butts" deviceset="RESISTOR" device="PTH-AXIAL-10.16MM" value="1R5"/>
 <part name="GND2" library="A_butts" deviceset="GND" device=""/>
 <part name="H1" library="A_butts" deviceset="HOLE" device="#2"/>
 <part name="H2" library="A_butts" deviceset="HOLE" device="#2"/>
-<part name="D1" library="A_butts" deviceset="DIODE-ZENER" device="PTH-7.62MM" value="10V"/>
+<part name="D1" library="A_butts" deviceset="DIODE-ZENER" device="10.16MM-PTH" value="10V"/>
 <part name="JP1" library="A_butts" deviceset="M04" device="PTH"/>
 <part name="IC1" library="A_butts" deviceset="ATTINY45" device="TINY85-20-DIP" value="TINY85-20-DIP"/>
@@
 <part name="SUPPLY3" library="A_butts" deviceset="VCC" device=""/>
 <part name="GND3" library="A_butts" deviceset="GND" device=""/>
-<part name="R1" library="A_butts" deviceset="RESISTOR" device="PTH-AXIAL-6.35MM" value="100k"/>
+<part name="R1" library="A_butts" deviceset="RESISTOR" device="PTH-AXIAL-10.16MM" value="100k"/>
 <part name="SUPPLY4" library="A_butts" deviceset="VCC" device=""/>
 <part name="SUPPLY5" library="A_butts" deviceset="VCC" device=""/>
@@
 <part name="SUPPLY1" library="A_butts" deviceset="VCC" device=""/>
 <part name="Q3" library="A_butts" deviceset="TRANSISTOR_NPN" device="TO-92-AMMO-EBC" value="2N3904"/>
-<part name="Q4" library="A_butts" deviceset="MOSFET-NCHANNEL" device="TO-220" value="IRLZ14PBF"/>
+<part name="Q4" library="A_butts" deviceset="MOSFET-NCHANNEL" device="TO-220" value="FQP30N06L"/>
 <part name="R3" library="A_butts" deviceset="RESISTOR" device="PTH-AXIAL-10.16MM" value="1R5"/>
 <part name="GND1" library="A_butts" deviceset="GND" device=""/>
-<part name="D2" library="A_butts" deviceset="DIODE-ZENER" device="PTH-7.62MM" value="10V"/>
+<part name="D2" library="A_butts" deviceset="DIODE-ZENER" device="10.16MM-PTH" value="10V"/>
 <part name="Q5" library="A_butts" deviceset="TRANSISTOR_NPN" device="TO-92-AMMO-EBC" value="2N3904"/>
-<part name="Q6" library="A_butts" deviceset="MOSFET-NCHANNEL" device="TO-220" value="IRLZ14PBF"/>
+<part name="Q6" library="A_butts" deviceset="MOSFET-NCHANNEL" device="TO-220" value="FQP30N06L"/>
 <part name="R4" library="A_butts" deviceset="RESISTOR" device="PTH-AXIAL-10.16MM" value="1R5"/>
 <part name="GND5" library="A_butts" deviceset="GND" device=""/>
-<part name="D3" library="A_butts" deviceset="DIODE-ZENER" device="PTH-7.62MM" value="10V"/>
+<part name="D3" library="A_butts" deviceset="DIODE-ZENER" device="10.16MM-PTH" value="10V"/>
 </parts>
 <sheets>
