File: hardware/just_a_switch-mk-2.0.brd (EAGLE design)
At the start: 22.9 x 17.8 mm, 13 parts, among them U1_ ROTARY_ENCODER_SWITCH, U2 Tiny85

Commit message: have some boards, dawg
Parts:
- removed A, B, GND, RST, SCL, SDA, SW, VCC: M01PTH-1MM, a_parts:1X01-1MM-NS
- removed C1: 100n, a_parts:C0603-TIGHTER
- removed FRAME1: FRAME-LETTERNO_PACKAGE, A_butts:DUMMY
- removed U1_: ROTARY_ENCODER_SWITCH, a_parts:ROTARY_ENCODER_SWITCH
- removed U2: Tiny85, a_parts:SO08-EIAJ
- added IN, OUT: M02PTH-CENTERED-R+, a_parts:1X02-CENTER-R+
- added LED1: LED3MM-LESS, A_butts:LED3MM-LESSSILK
- added PWR: SWITCH-SPSTROCKER, a_parts:SPST-ROCKER-3.81MM
- added Q1: 2N7000, A_butts:TO-92-AMMO
- added R2: 10K, A_butts:RESISTOR-AXIAL-PTH-5.08MM
- R1: device a_parts:R0603-TIGHTER -> A_butts:RESISTOR-AXIAL-PTH-5.08MM
- moved R1 4.33 mm to (9.00, 10.0), flipped to the top, turned to 0 degrees
Connections:
- removed net A: A.1, U1_.A, U2.3
- removed net B: B.1, U1_.B, U2.2
- removed net MOSI/SDA: SDA.1, U2.5
- removed net RST: R1.1, RST.1, U2.1
- removed net SCK/SCL: SCL.1, U2.7
- removed net SW: SW.1, U1_.SW1, U2.6
- new net GND_IN: LED1.K, OUT.1, Q1.3
- new net N$1: IN.2, PWR.COM
- new net N$2: LED1.A, R2.P$1
- net GND: now also IN.1, Q1.1, R1.P$1; no longer C1.2, GND.1, U1_.C, U1_.SW2, U2.4
- net VCC: now also OUT.2, PWR.NO, Q1.2, R1.P$2, R2.P$2; no longer C1.1, R1.2, U2.8, VCC.1
Routing:
- net SW: track 22.5 -> 0.00 mm, vias 1 -> 0
- net VCC: track 17.0 -> 0.00 mm
- net RST: track 10.5 -> 0.00 mm
- net B: track 9.54 -> 0.00 mm
- net MOSI/SDA: track 7.77 -> 0.00 mm
- net A: track 7.74 -> 0.00 mm
- net SCK/SCL: track 7.25 -> 0.00 mm
- removed copper zone on layer 16, net GND
Other:
- board size 22.9 x 17.8 mm -> 24 x 15 mm
- board text removed: ">VERSION"
- board text removed: "A"
- board text removed: "B"
- board text removed: "C"
- board text removed: "COM"
- board text removed: "ENCODIFIER"
- board text removed: "SW"
