File: hardware/rev-polarity-deflector-dish-mk-1.0.brd (EAGLE design)
At the start: 22.9 x 17.8 mm, 13 parts, among them U1_ ROTARY_ENCODER_SWITCH, U2 Tiny85

Commit message: have some boards, dawg
Parts:
- removed A, B, GND, RST, SCL, SDA, SW, VCC: M01PTH-1MM, a_parts:1X01-1MM-NS
- removed C1: 100n, a_parts:C0603-TIGHTER
- removed U1_: ROTARY_ENCODER_SWITCH, a_parts:ROTARY_ENCODER_SWITCH
- removed U2: Tiny85, a_parts:SO08-EIAJ
- added D1: 1N4740, a_parts:DIODE-ZENNER-7.62MM
- added IN, OUT: M02PTH-CENTERED-R+, a_parts:1X02-CENTER-R+
- added LED1: LED3MM-LESS, a_parts:LED3MM-LESSSILK
- added PWR: SWITCH-SPDTPTH-VERT-2.54MM, a_parts:SWITCH-SPDT
- added Q1: 2N7000, a_parts:TO-92-AMMO
- added R2, R3: 10K, a_parts:RESISTOR-AXIAL-PTH-7.62MM
- R1: value 10k -> 10K; device a_parts:R0603-TIGHTER -> a_parts:RESISTOR-AXIAL-PTH-7.62MM
- moved R1 29.6 mm to (38.0, 11.0), flipped to the top, turned to 90 degrees
Connections:
- removed net A: A.1, U1_.A, U2.3
- removed net B: B.1, U1_.B, U2.2
- removed net GND: C1.2, GND.1, U1_.C, U1_.SW2, U2.4
- removed net MOSI/SDA: SDA.1, U2.5
- removed net RST: R1.1, RST.1, U2.1
- removed net SCK/SCL: SCL.1, U2.7
- removed net SW: SW.1, U1_.SW1, U2.6
- removed net VCC: C1.1, R1.2, U2.8, VCC.1
- new net N$1: D1.K, Q1.2, R1.P$2
- new net N$2: LED1.K, R3.P$2
- new net VIN+: IN.2, PWR.2
- new net VIN-: D1.A, IN.1, Q1.1, R2.P$2
- new net VOUT+: OUT.2, PWR.3, R1.P$1, R2.P$1, R3.P$1
- new net VOUT-: LED1.A, OUT.1, Q1.3
Routing:
- net SW: track 22.5 -> 0.00 mm, vias 1 -> 0
- net VCC: track 17.0 -> 0.00 mm
- net RST: track 10.5 -> 0.00 mm
- net B: track 9.54 -> 0.00 mm
- net MOSI/SDA: track 7.77 -> 0.00 mm
- net A: track 7.74 -> 0.00 mm
- net SCK/SCL: track 7.25 -> 0.00 mm
- added copper zone on layer 16, net VIN-
- added copper zone on layer 1, net VOUT-
- removed copper zone on layer 1, net GND
- removed copper zone on layer 16, net GND
Other:
- board size 22.9 x 17.8 mm -> 20 x 20 mm
- board text removed: ">VERSION"
- board text removed: "A"
- board text removed: "B"
- board text removed: "C"
- board text removed: "COM"
- board text removed: "ENCODIFIER"
- board text removed: "SW"
